Commit message: 231212

File: z1_description/xacro/z1_arm.xacro (robot description, xacro)
@@ -135,283 +135,330 @@
   <xacro:property name="gripperBox_Y" value="0."/>
   <xacro:property name="gripperBox_Z" value="0."/>
-  <xacro:arg name="UnitreeGripper" default="false"/>
-  <!-- Define Link and Joints of the Unitree Z1_arm -->
-  <link name="base_link"/>
+  <!-- About Gripper -->
+  <xacro:arg name="UnitreeGripper" default="true"/>
+  <!-- Transmission macro -->
+  <xacro:macro name="motorTransmission" params="name">
+    <transmission name="JointTrans${name}">
+      <type>transmission_interface/SimpleTransmission</type>
+      <joint name="joint${name}">
+        <hardwareInterface>hardware_interface/EffortJointInterface</hardwareInterface>
+      </joint>
+      <actuator name="Actuator${name}">
+        <hardwareInterface>hardware_interface/EffortJointInterface</hardwareInterface>
+        <mechanicalReduction>1</mechanicalReduction>
+      </actuator>
+    </transmission>
+  </xacro:macro>
+  <!-- Bottom Fixed Link
+  This link is the base of the arm where arm is placed
+  -->
+  <!-- ////////////////////////////////////////////////////////////////////////////////////////////////////////// -->
+  <link name="world"/>
   <joint name="base_static_joint" type="fixed">
-  <origin rpy="0 0 0" xyz="0 0 0"/>
-  <parent link="base_link"/>
-  <child link="link00"/>
-  </joint>
+      <origin rpy="0 0 0" xyz="0 0 0"/>
+      <parent link="world"/>
+      <child link="link00"/>
+  </joint>
+  <!-- ////////////////////////////////////////////////////////////////////////////////////////////////////////////-->
+  <!-- LINK 00 -->
   <link name="link00">
-  <visual>
-  <origin rpy="0 0 0" xyz="0 0 0"/>
-  <geometry>
-      <mesh filename="package://z1_description/meshes/visual/z1_Link00.dae" scale="1 1 1"/>
-  </geometry>
-  </visual>
-  <collision>
-  <geometry>
-      <cylinder length="${motor_height}" radius="${motor_diameter}"/>
-  </geometry>
-  <origin rpy="0 0 0" xyz="0 0 ${motor_height/2.0}"/>
-  </collision>
-  <inertial>
-  <origin rpy="0 0 0" xyz="${L00_ComX} ${L00_ComY} ${L00_ComZ}"/>
-  <mass value="${L00_Mass}"/>
-  <inertia
-      ixx="${L00_Ixx}" ixy="${L00_Ixy}" ixz="${L00_Ixz}"
-      iyy="${L00_Iyy}" iyz="${L00_Iyz}"
-      izz="${L00_Izz}"/>
-  </inertial>
+      <visual>
+          <origin rpy="0 0 0" xyz="0 0 0"/>
+          <geometry>
+              <mesh filename="package://z1_description/meshes/visual/z1_Link00.dae" scale="1 1 1"/>
+          </geometry>
+      </visual>
+      <collision>
+          <geometry>
+              <cylinder length="${motor_height}" radius="${motor_diameter}"/>
+          </geometry>
+          <origin rpy="0 0 0" xyz="0 0 ${motor_height/2.0}"/>
+      </collision>
+      <inertial>
+          <origin rpy="0 0 0" xyz="${L00_ComX} ${L00_ComY} ${L00_ComZ}"/>
+          <mass value="${L00_Mass}"/>
+          <inertia
+              ixx="${L00_Ixx}" ixy="${L00_Ixy}" ixz="${L00_Ixz}"
+              iyy="${L00_Iyy}" iyz="${L00_Iyz}"
+              izz="${L00_Izz}"/>
+      </inertial>
   </link>
   <joint name="joint1" type="revolute">
-  <origin rpy="0 0 0" xyz="0 0 0.0585"/>
-  <parent link="link00"/>
-  <child link="link01"/>
-  <axis xyz="0 0 1"/>
-  <dynamics damping="${jointDamping}" friction="${jointFriction}"/>
-  <limit effort="${torqueMax}" velocity="${velocityMax}" lower="${joint1_PositionMin}" upper="${joint1_PositionMax}"/>
-  </joint>
+      <origin rpy="0 0 0" xyz="0 0 0.0585"/>
+      <parent link="link00"/>
+      <child link="link01"/>
+      <axis xyz="0 0 1"/>
+      <dynamics damping="${jointDamping}" friction="${jointFriction}"/>
+      <limit effort="${torqueMax}" velocity="${velocityMax}" lower="${joint1_PositionMin}" upper="${joint1_PositionMax}"/>
+  </joint>
+  <!-- ////////////////////////////////////////////////////////////////////////////////////////////////////////////-->
+  <!-- LINK 01 -->
   <link name="link01">
-  <visual>
-  <origin rpy="0 0 0" xyz="0 0 0"/>
-  <geometry>
-      <mesh filename="package://z1_description/meshes/visual/z1_Link01.dae" scale="1 1 1"/>
-  </geometry>
-  </visual>
-  <inertial>
-  <origin rpy="0 0 0" xyz="${L01_ComX} ${L01_ComY} ${L01_ComZ}"/>
-  <mass value="${L01_Mass}"/>
-  <inertia
-      ixx="${L01_Ixx}" ixy="${L01_Ixy}" ixz="${L01_Ixz}"
-      iyy="${L01_Iyy}" iyz="${L01_Iyz}"
-      izz="${L01_Izz}"/>
-  </inertial>
+      <visual>
+          <origin rpy="0 0 0" xyz="0 0 0"/>
+          <geometry>
+              <mesh filename="package://z1_description/meshes/visual/z1_Link01.dae" scale="1 1 1"/>
+          </geometry>
+      </visual>
+      <inertial>
+          <origin rpy="0 0 0" xyz="${L01_ComX} ${L01_ComY} ${L01_ComZ}"/>
+          <mass value="${L01_Mass}"/>
+          <inertia
+              ixx="${L01_Ixx}" ixy="${L01_Ixy}" ixz="${L01_Ixz}"
+              iyy="${L01_Iyy}" iyz="${L01_Iyz}"
+              izz="${L01_Izz}"/>
+      </inertial>
   </link>
   <joint name="joint2" type="revolute">
-  <origin rpy="0 0 0" xyz="0 0 0.045"/>
-  <parent link="link01"/>
-  <child link="link02"/>
-  <axis xyz="0 1 0"/>
-  <dynamics damping="${2*jointDamping}" friction="${2*jointFriction}"/>
-  <limit effort="${2*torqueMax}" velocity="${velocityMax}" lower="${joint2_PositionMin}" upper="${joint2_PositionMax}"/>
-  </joint>
+      <origin rpy="0 0 0" xyz="0 0 0.045"/>
+      <parent link="link01"/>
+      <child link="link02"/>
+      <axis xyz="0 1 0"/>
+      <dynamics damping="${2*jointDamping}" friction="${2*jointFriction}"/>
+      <limit effort="${2*torqueMax}" velocity="${velocityMax}" lower="${joint2_PositionMin}" upper="${joint2_PositionMax}"/>
+  </joint>
+  <!-- ////////////////////////////////////////////////////////////////////////////////////////////////////////////-->
+  <!-- LINK 02 -->
   <link name="link02">
-  <visual>
-  <origin rpy="0 0 0" xyz="0 0 0"/>
-  <geometry>
-      <mesh filename="package://z1_description/meshes/visual/z1_Link02.dae" scale="1 1 1"/>
-  </geometry>
-  </visual>
-  <collision>
-  <geometry>
-      <cylinder length="${2.0*motor_height}" radius="${motor_diameter}"/>
-  </geometry>
-  <origin rpy="${PI/2.0} 0 0" xyz="0 0 0"/>
-  </collision>
-  <collision>
-  <geometry>
-      <cylinder length="${arm1_height}" radius="${arm1_diameter}"/>
-  </geometry>
-  <origin rpy="0 ${PI/2.0} 0" xyz="${-0.045-arm1_height/2.0} 0 0"/>
-  </collision>
-  <collision>
-  <geometry>
-      <cylinder length="${motor_height}" radius="${motor_diameter}"/>
-  </geometry>
-  <origin rpy="${PI/2.0} 0 0" xyz="-0.35 0 0"/>
-  </collision>
-  <inertial>
-  <origin rpy="0 0 0" xyz="${L02_ComX} ${L02_ComY} ${L02_ComZ}"/>
-  <mass value="${L02_Mass}"/>
-  <inertia
-      ixx="${L02_Ixx}" ixy="${L02_Ixy}" ixz="${L02_Ixz}"
-      iyy="${L02_Iyy}" iyz="${L02_Iyz}"
-      izz="${L02_Izz}"/>
-  </inertial>
+      <visual>
+          <origin rpy="0 0 0" xyz="0 0 0"/>
+          <geometry>
+              <mesh filename="package://z1_description/meshes/visual/z1_Link02.dae" scale="1 1 1"/>
+          </geometry>
+      </visual>
+      <collision>
+          <geometry>
+              <cylinder length="${2.0*motor_height}" radius="${motor_diameter}"/>
+          </geometry>
+          <origin rpy="${PI/2.0} 0 0" xyz="0 0 0"/>
+      </collision>
+      <collision>
+          <geometry>
+              <cylinder length="${arm1_height}" radius="${arm1_diameter}"/>
+          </geometry>
+          <origin rpy="0 ${PI/2.0} 0" xyz="${-0.045-arm1_height/2.0} 0 0"/>
+      </collision>
+      <collision>
+          <geometry>
+              <cylinder length="${motor_height}" radius="${motor_diameter}"/>
+          </geometry>
+          <origin rpy="${PI/2.0} 0 0" xyz="-0.35 0 0"/>
+      </collision>
+      <inertial>
+          <origin rpy="0 0 0" xyz="${L02_ComX} ${L02_ComY} ${L02_ComZ}"/>
+          <mass value="${L02_Mass}"/>
+          <inertia
+              ixx="${L02_Ixx}" ixy="${L02_Ixy}" ixz="${L02_Ixz}"
+              iyy="${L02_Iyy}" iyz="${L02_Iyz}"
+              izz="${L02_Izz}"/>
+      </inertial>
   </link>
   <joint name="joint3" type="revolute">
-  <origin rpy="0 0 0" xyz="-0.35 0 0"/>
-  <parent link="link02"/>
-  <child link="link03"/>
-  <axis xyz="0 1 0"/>
-  <dynamics damping="${jointDamping}" friction="${jointFriction}"/>
-  <limit effort="${torqueMax}" velocity="${velocityMax}" lower="${joint3_PositionMin}" upper="${joint3_PositionMax}"/>
-  </joint>
+      <origin rpy="0 0 0" xyz="-0.35 0 0"/>
+      <parent link="link02"/>
+      <child link="link03"/>
+      <axis xyz="0 1 0"/>
+      <dynamics damping="${jointDamping}" friction="${jointFriction}"/>
+      <limit effort="${torqueMax}" velocity="${velocityMax}" lower="${joint3_PositionMin}" upper="${joint3_PositionMax}"/>
+  </joint>
+  <!-- ////////////////////////////////////////////////////////////////////////////////////////////////////////////-->
+  <!-- LINK 03 -->
   <link name="link03">
-  <visual>
-  <origin rpy="0 0 0" xyz="0 0 0"/>
-  <geometry>
-      <mesh filename="package://z1_description/meshes/visual/z1_Link03.dae" scale="1 1 1"/>
-  </geometry>
-  </visual>
-  <collision>
-  <geometry>
-      <cylinder length="${arm2_height-0.01}" radius="${arm2_diameter}"/>
-  </geometry>
-  <origin rpy="0 ${PI/2.0} 0" xyz="${0.065+arm2_height/2.0} 0 0.055"/>
-  </collision>
-  <collision>
-  <geometry>
-      <cylinder length="0.059" radius="${motor_diameter}"/>
-  </geometry>
-  <origin rpy="0 ${PI/2.0} ${PI/2.0}" xyz="${0.065+0.185-0.059/2.0} 0 0.055"/>
-  </collision>
-  <inertial>
-  <origin rpy="0 0 0" xyz="${L03_ComX} ${L03_ComY} ${L03_ComZ}"/>
-  <mass value="${L03_Mass}"/>
-  <inertia
-      ixx="${L03_Ixx}" ixy="${L03_Ixy}" ixz="${L03_Ixz}"
-      iyy="${L03_Iyy}" iyz="${L03_Iyz}"
-      izz="${L03_Izz}"/>
-  </inertial>
+      <visual>
+          <origin rpy="0 0 0" xyz="0 0 0"/>
+          <geometry>
+              <mesh filename="package://z1_description/meshes/visual/z1_Link03.dae" scale="1 1 1"/>
+          </geometry>
+      </visual>
+      <collision>
+          <geometry>
+              <cylinder length="${arm2_height-0.01}" radius="${arm2_diameter}"/>
+          </geometry>
+          <origin rpy="0 ${PI/2.0} 0" xyz="${0.065+arm2_height/2.0} 0 0.055"/>
+      </collision>
+      <collision>
+          <geometry>
+              <cylinder length="0.059" radius="${motor_diameter}"/>
+          </geometry>
+          <origin rpy="0 ${PI/2.0} ${PI/2.0}" xyz="${0.065+0.185-0.059/2.0} 0 0.055"/>
+      </collision>
+      <inertial>
+          <origin rpy="0 0 0" xyz="${L03_ComX} ${L03_ComY} ${L03_ComZ}"/>
+          <mass value="${L03_Mass}"/>
+          <inertia
+              ixx="${L03_Ixx}" ixy="${L03_Ixy}" ixz="${L03_Ixz}"
+              iyy="${L03_Iyy}" iyz="${L03_Iyz}"
+              izz="${L03_Izz}"/>
+      </inertial>
   </link>
   <joint name="joint4" type="revolute">
-  <origin rpy="0 0 0" xyz="0.218 0 0.057"/>
-  <parent link="link03"/>
-  <child link="link04"/>
-  <axis xyz="0 1 0"/>
-  <dynamics damping="${jointDamping}" friction="${jointFriction}"/>
-  <limit effort="${torqueMax}" velocity="${velocityMax}" lower="${joint4_PositionMin}" upper="${joint4_PositionMax}"/>
-  </joint>
+      <origin rpy="0 0 0" xyz="0.218 0 0.057"/>
+      <parent link="link03"/>
+      <child link="link04"/>
+      <axis xyz="0 1 0"/>
+      <dynamics damping="${jointDamping}" friction="${jointFriction}"/>
+      <limit effort="${torqueMax}" velocity="${velocityMax}" lower="${joint4_PositionMin}" upper="${joint4_PositionMax}"/>
+  </joint>
+  <!-- ////////////////////////////////////////////////////////////////////////////////////////////////////////////-->
+  <!-- LINK 04 -->
   <link name="link04">
-  <visual>
-  <origin rpy="0 0 0" xyz="0 0 0"/>
-  <geometry>
-      <mesh filename="package://z1_description/meshes/visual/z1_Link04.dae" scale="1 1 1"/>
-  </geometry>
-  </visual>
-  <collision>
-  <geometry>
-      <cylinder length="${motor_height + 2*0.008}" radius="${motor_diameter}"/>
-  </geometry>
-  <origin rpy="0 0 0" xyz="0.072 0 0"/>
-  </collision>
-  <inertial>
-  <origin rpy="0 0 0" xyz="${L04_ComX} ${L04_ComY} ${L04_ComZ}"/>
-  <mass value="${L04_Mass}"/>
-  <inertia
-      ixx="${L04_Ixx}" ixy="${L04_Ixy}" ixz="${L04_Ixz}"
-      iyy="${L04_Iyy}" iyz="${L04_Iyz}"
-      izz="${L04_Izz}"/>
-  </inertial>
-  </link>
+      <visual>
+          <origin rpy="0 0 0" xyz="0 0 0"/>
+          <geometry>
+              <mesh filename="package://z1_description/meshes/visual/z1_Link04.dae" scale="1 1 1"/>
+          </geometry>
+      </visual>
+      <collision>
+          <geometry>
+              <cylinder length="${motor_height + 2*0.008}" radius="${motor_diameter}"/>
+          </geometry>
+          <origin rpy="0 0 0" xyz="0.072 0 0"/>
+      </collision>
+      <inertial>
+          <origin rpy="0 0 0" xyz="${L04_ComX} ${L04_ComY} ${L04_ComZ}"/>
+          <mass value="${L04_Mass}"/>
+          <inertia
+              ixx="${L04_Ixx}" ixy="${L04_Ixy}" ixz="${L04_Ixz}"
+              iyy="${L04_Iyy}" iyz="${L04_Iyz}"
+              izz="${L04_Izz}"/>
+      </inertial>
+  </link>
+  <gazebo reference="link04">
+    <self_collide>true</self_collide>
+  </gazebo>
   <joint name="joint5" type="revolute">
-  <origin rpy="0 0 0" xyz="0.07 0.0 0.0"/>
-  <parent link="link04"/>
-  <child link="link05"/>
-  <axis xyz="0 0 1"/>
-  <dynamics damping="${jointDamping}" friction="${jointFriction}"/>
-  <limit effort="${torqueMax}" velocity="${velocityMax}" lower="${joint5_PositionMin}" upper="${joint5_PositionMax}"/>
-  </joint>
+      <origin rpy="0 0 0" xyz="0.07 0.0 0.0"/>
+      <parent link="link04"/>
+      <child link="link05"/>
+      <axis xyz="0 0 1"/>
+      <dynamics damping="${jointDamping}" friction="${jointFriction}"/>
+      <limit effort="${torqueMax}" velocity="${velocityMax}" lower="${joint5_PositionMin}" upper="${joint5_PositionMax}"/>
+  </joint>
+  <!-- ////////////////////////////////////////////////////////////////////////////////////////////////////////////-->
+  <!-- LINK 05 -->
   <link name="link05">
-  <visual>
-  <origin rpy="0 0 0" xyz="0 0 0"/>
-  <geometry>
-      <mesh filename="package://z1_description/meshes/visual/z1_Link05.dae" scale="1 1 1"/>
-  </geometry>
-  </visual>
-  <inertial>
-  <origin rpy="0 0 0" xyz="${L05_ComX} ${L05_ComY} ${L05_ComZ}"/>
-  <mass value="${L05_Mass}"/>
-  <inertia
-      ixx="${L05_Ixx}" ixy="${L05_Ixy}" ixz="${L05_Ixz}"
-      iyy="${L05_Iyy}" iyz="${L05_Iyz}"
-      izz="${L05_Izz}"/>
-  </inertial>
-  </link>
+      <visual>
+          <origin rpy="0 0 0" xyz="0 0 0"/>
+          <geometry>
+              <mesh filename="package://z1_description/meshes/visual/z1_Link05.dae" scale="1 1 1"/>
+          </geometry>
+      </visual>
+      <inertial>
+          <origin rpy="0 0 0" xyz="${L05_ComX} ${L05_ComY} ${L05_ComZ}"/>
+          <mass value="${L05_Mass}"/>
+          <inertia
+              ixx="${L05_Ixx}" ixy="${L05_Ixy}" ixz="${L05_Ixz}"
+              iyy="${L05_Iyy}" iyz="${L05_Iyz}"
+              izz="${L05_Izz}"/>
+      </inertial>
+  </link>
+  <gazebo reference="link05">
+      <self_collide>true</self_collide>
+  </gazebo>
   <joint name="joint6" type="revolute">
-  <origin rpy="0 0 0" xyz="0.0492 0.0 0.0"/>
-  <parent link="link05"/>
-  <child link="link06"/>
-  <axis xyz="1 0 0"/>
-  <dynamics damping="${jointDamping}" friction="${jointFriction}"/>
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